Commit message: bf presentation

File: install/ros2_control_demo_description/share/ros2_control_demo_description/rrbot/urdf/rrbot_description.urdf.xacro (robot description, xacro)
@@ -5,7 +5,7 @@
   <xacro:property name="mass" value="1" /> <!-- arbitrary value for mass -->
   <xacro:property name="width" value="0.1" /> <!-- Square dimensions (widthxwidth) of beams -->
-  <xacro:property name="height1" value="1" /> <!-- Link 1 -->
-  <xacro:property name="height2" value="0.5" /> <!-- Link 2 -->
-  <xacro:property name="height3" value="0.5" /> <!-- Link 3 -->
+  <xacro:property name="height1" value="2" /> <!-- Link 1 -->
+  <xacro:property name="height2" value="1" /> <!-- Link 2 -->
+  <xacro:property name="height3" value="1" /> <!-- Link 3 -->
   <xacro:property name="axel_offset" value="0.05" /> <!-- Space btw top of beam and the each joint -->
   <joint name="${prefix}base_joint" type="fixed">
@@ -25,5 +25,5 @@
       <origin xyz="0 0 ${height1/2}" rpy="0 0 0"/>
       <geometry>
-        <box size="${width} ${width} ${height1}"/>
+        <box size="${width*4} ${width*10} ${height1}"/>
       </geometry>
       <material name="blue"/>
@@ -100,7 +100,69 @@
     </inertial>
   </link>
+  <!-- Middle Link 2-->
+  <link name="${prefix}link3">
+    <collision>
+      <origin xyz="0 0 ${height2/2 - axel_offset}" rpy="0 0 0"/>
+      <geometry>
+        <box size="${width} ${width} ${height2}"/>
+      </geometry>
+    </collision>
+    <visual>
+      <origin xyz="0 0 ${height2/2 - axel_offset}" rpy="0 0 0"/>
+      <geometry>
+        <box size="${width} ${width} ${height2}"/>
+      </geometry>
+      <material name="red"/>
+    </visual>
+    <inertial>
+      <origin xyz="0 0 ${height2/2 - axel_offset}" rpy="0 0 0"/>
+      <mass value="${mass}"/>
+      <inertia
+        ixx="${mass / 12.0 * (width*width + height2*height2)}" ixy="0.0" ixz="0.0"
+        iyy="${mass / 12.0 * (height2*height2 + width*width)}" iyz="0.0"
+        izz="${mass / 12.0 * (width*width + width*width)}"/>
+    </inertial>
+  </link>
+  <joint name="${prefix}joint3" type="continuous">
+    <parent link="${prefix}base_link"/>
+    <child link="${prefix}link3"/>
+    <origin xyz="0 ${width+0.5} ${height1 - axel_offset}" rpy="0 0 0"/>
+    <axis xyz="0 1 0"/>
+    <dynamics damping="0.7"/>
+  </joint>
+  <!-- Top Link 2-->
+  <link name="${prefix}link4">
+    <collision>
+      <origin xyz="0 0 ${height3/2 - axel_offset}" rpy="0 0 0"/>
+      <geometry>
+        <box size="${width} ${width} ${height3}"/>
+      </geometry>
+    </collision>
+    <visual>
+      <origin xyz="0 0 ${height3/2 - axel_offset}" rpy="0 0 0"/>
+      <geometry>
+        <box size="${width} ${width} ${height3}"/>
+      </geometry>
+      <material name="orange"/>
+    </visual>
+    <inertial>
+      <origin xyz="0 0 ${height3/2 - axel_offset}" rpy="0 0 0"/>
+      <mass value="${mass}"/>
+      <inertia
+        ixx="${mass / 12.0 * (width*width + height3*height3)}" ixy="0.0" ixz="0.0"
+        iyy="${mass / 12.0 * (height3*height3 + width*width)}" iyz="0.0"
+        izz="${mass / 12.0 * (width*width + width*width)}"/>
+    </inertial>
+  </link>
+  <joint name="${prefix}joint4" type="continuous">
+    <parent link="${prefix}link3"/>
+    <child link="${prefix}link4"/>
+    <origin xyz="0 ${width} ${height2 - axel_offset}" rpy="0 0 0"/>
+    <axis xyz="0 1 0"/>
+    <dynamics damping="0.7"/>
+  </joint>
   <joint name="${prefix}tool_joint" type="fixed">
     <origin xyz="0 0 1" rpy="0 0 0" />
-    <parent link="${prefix}link2"/>
+    <parent link="${prefix}link3"/>
     <child link="${prefix}tool_link" />
   </joint>

File: src/ros2_control_demo_description/rrbot/urdf/rrbot_description.urdf.xacro (robot description, xacro)
@@ -25,5 +25,5 @@
       <origin xyz="0 0 ${height1/2}" rpy="0 0 0"/>
       <geometry>
-        <box size="${width} ${width} ${height1}"/>
+        <box size="${width*4} ${width*10} ${height1}"/>
       </geometry>
       <material name="blue"/>
@@ -100,7 +100,69 @@
     </inertial>
   </link>
+  <!-- Middle Link 2-->
+  <link name="${prefix}link3">
+    <collision>
+      <origin xyz="0 0 ${height2/2 - axel_offset}" rpy="0 0 0"/>
+      <geometry>
+        <box size="${width} ${width} ${height2}"/>
+      </geometry>
+    </collision>
+    <visual>
+      <origin xyz="0 0 ${height2/2 - axel_offset}" rpy="0 0 0"/>
+      <geometry>
+        <box size="${width} ${width} ${height2}"/>
+      </geometry>
+      <material name="red"/>
+    </visual>
+    <inertial>
+      <origin xyz="0 0 ${height2/2 - axel_offset}" rpy="0 0 0"/>
+      <mass value="${mass}"/>
+      <inertia
+        ixx="${mass / 12.0 * (width*width + height2*height2)}" ixy="0.0" ixz="0.0"
+        iyy="${mass / 12.0 * (height2*height2 + width*width)}" iyz="0.0"
+        izz="${mass / 12.0 * (width*width + width*width)}"/>
+    </inertial>
+  </link>
+  <joint name="${prefix}joint3" type="continuous">
+    <parent link="${prefix}base_link"/>
+    <child link="${prefix}link3"/>
+    <origin xyz="0 ${width+0.5} ${height1 - axel_offset}" rpy="0 0 0"/>
+    <axis xyz="0 1 0"/>
+    <dynamics damping="0.7"/>
+  </joint>
+  <!-- Top Link 2-->
+  <link name="${prefix}link4">
+    <collision>
+      <origin xyz="0 0 ${height3/2 - axel_offset}" rpy="0 0 0"/>
+      <geometry>
+        <box size="${width} ${width} ${height3}"/>
+      </geometry>
+    </collision>
+    <visual>
+      <origin xyz="0 0 ${height3/2 - axel_offset}" rpy="0 0 0"/>
+      <geometry>
+        <box size="${width} ${width} ${height3}"/>
+      </geometry>
+      <material name="orange"/>
+    </visual>
+    <inertial>
+      <origin xyz="0 0 ${height3/2 - axel_offset}" rpy="0 0 0"/>
+      <mass value="${mass}"/>
+      <inertia
+        ixx="${mass / 12.0 * (width*width + height3*height3)}" ixy="0.0" ixz="0.0"
+        iyy="${mass / 12.0 * (height3*height3 + width*width)}" iyz="0.0"
+        izz="${mass / 12.0 * (width*width + width*width)}"/>
+    </inertial>
+  </link>
+  <joint name="${prefix}joint4" type="continuous">
+    <parent link="${prefix}link3"/>
+    <child link="${prefix}link4"/>
+    <origin xyz="0 ${width} ${height2 - axel_offset}" rpy="0 0 0"/>
+    <axis xyz="0 1 0"/>
+    <dynamics damping="0.7"/>
+  </joint>
   <joint name="${prefix}tool_joint" type="fixed">
     <origin xyz="0 0 1" rpy="0 0 0" />
-    <parent link="${prefix}link2"/>
+    <parent link="${prefix}link3"/>
     <child link="${prefix}tool_link" />
   </joint>

File: src/ros2_control_hand/description/ros2_control/rrbot.ros2_control.xacro (robot description, xacro)
@@ -20,4 +20,18 @@
         <state_interface name="position"/>
       </joint>
+      <joint name="${prefix}joint3">
+        <command_interface name="position">
+          <param name="min">-1</param>
+          <param name="max">1</param>
+        </command_interface>
+        <state_interface name="position"/>
+      </joint>
+      <joint name="${prefix}joint4">
+        <command_interface name="position">
+          <param name="min">-1</param>
+          <param name="max">1</param>
+        </command_interface>
+        <state_interface name="position"/>
+      </joint>
     </ros2_control>
   </xacro:macro>

Commit message: added 3 fingers

File: install/ros2_control_demo_description/share/ros2_control_demo_description/rrbot/urdf/rrbot_description.urdf.xacro (robot description, xacro)
@@ -3,10 +3,9 @@
   <xacro:macro name="rrbot" params="parent prefix *origin">
   <!-- Constants for robot dimensions -->
-  <xacro:property name="mass" value="1" /> <!-- arbitrary value for mass -->
+  <xacro:property name="mass" value="1" /> <!-- Arbitrary value for mass -->
   <xacro:property name="width" value="0.1" /> <!-- Square dimensions (widthxwidth) of beams -->
-  <xacro:property name="height1" value="2" /> <!-- Link 1 -->
-  <xacro:property name="height2" value="1" /> <!-- Link 2 -->
-  <xacro:property name="height3" value="1" /> <!-- Link 3 -->
-  <xacro:property name="axel_offset" value="0.05" /> <!-- Space btw top of beam and the each joint -->
+  <xacro:property name="height1" value="2" /> <!-- Length of finger base -->
+  <xacro:property name="height2" value="1" /> <!-- Length of middle finger segment -->
+  <xacro:property name="axel_offset" value="0.05" /> <!-- Space between top of beam and each joint -->
   <joint name="${prefix}base_joint" type="fixed">
     <xacro:insert_block name="origin" />
@@ -38,19 +37,53 @@
     </inertial>
   </link>
-  <joint name="${prefix}joint1" type="continuous">
-    <parent link="${prefix}base_link"/>
-    <child link="${prefix}link1"/>
+  <!-- Finger 1 Base Link -->
+  <link name="${prefix}finger1_base">
+    <!-- Collision properties -->
+    <collision>
+      <origin xyz="0 0 ${height1/2}" rpy="0 0 0"/>
+      <geometry>
+        <box size="${width} ${width} ${height1}"/>
+      </geometry>
+    </collision>
+    <!-- Visual properties -->
+    <visual>
+      <origin xyz="0 0 ${height1/2}" rpy="0 0 0"/>
+      <geometry>
+        <box size="${width*4} ${width*10} ${height1}"/>
+      </geometry>
+      <material name="blue"/>
+    </visual>
+    <!-- Inertial properties -->
+    <inertial>
+      <origin xyz="0 0 ${height1/2}" rpy="0 0 0"/>
+      <mass value="${mass}"/>
+      <inertia
+        ixx="${mass / 12.0 * (width*width + height1*height1)}" ixy="0.0" ixz="0.0"
+        iyy="${mass / 12.0 * (height1*height1 + width*width)}" iyz="0.0"
+        izz="${mass / 12.0 * (width*width + width*width)}"/>
+    </inertial>
+  </link>
+  <!-- Joint for Finger 1 -->
+  <joint name="${prefix}joint_finger1" type="revolute">
+    <parent link="${prefix}base_link"/> <!-- Link to which the joint is connected -->
+    <child link="${prefix}finger1_base"/> <!-- Link that the joint connects to -->
+    <!-- Joint origin and axis -->
     <origin xyz="0 ${width} ${height1 - axel_offset}" rpy="0 0 0"/>
     <axis xyz="0 1 0"/>
-    <dynamics damping="0.7"/>
-  </joint>
-  <!-- Middle Link -->
-  <link name="${prefix}link1">
-    <collision>
-      <origin xyz="0 0 ${height2/2 - axel_offset}" rpy="0 0 0"/>
-      <geometry>
-        <box size="${width} ${width} ${height2}"/>
-      </geometry>
-    </collision>
+    <!-- Joint dynamics (optional) -->
+    <dynamics damping="0.7"/>
+    <!-- Joint limits -->
+    <limit effort="100" velocity="1.0" lower="-3.14" upper="3.14"/>
+  </joint>
+  <!-- Finger 1 Middle Link -->
+  <link name="${prefix}finger1_middle">
+    <!-- Collision properties -->
+    <collision>
+      <origin xyz="0 0 ${height2/2 - axel_offset}" rpy="0 0 0"/>
+      <geometry>
+        <box size="${width} ${width} ${height2}"/>
+      </geometry>
+    </collision>
+    <!-- Visual properties -->
     <visual>
       <origin xyz="0 0 ${height2/2 - axel_offset}" rpy="0 0 0"/>
@@ -60,4 +93,5 @@
       <material name="yellow"/>
     </visual>
+    <!-- Inertial properties -->
     <inertial>
       <origin xyz="0 0 ${height2/2 - axel_offset}" rpy="0 0 0"/>
@@ -69,50 +103,73 @@
     </inertial>
   </link>
-  <joint name="${prefix}joint2" type="continuous">
-    <parent link="${prefix}link1"/>
-    <child link="${prefix}link2"/>
-    <origin xyz="0 ${width} ${height2 - axel_offset*2}" rpy="0 0 0"/>
-    <axis xyz="0 1 0"/>
-    <dynamics damping="0.7"/>
-  </joint>
-  <!-- Top Link -->
-  <link name="${prefix}link2">
-    <collision>
-      <origin xyz="0 0 ${height3/2 - axel_offset}" rpy="0 0 0"/>
-      <geometry>
-        <box size="${width} ${width} ${height3}"/>
-      </geometry>
-    </collision>
-    <visual>
-      <origin xyz="0 0 ${height3/2 - axel_offset}" rpy="0 0 0"/>
-      <geometry>
-        <box size="${width} ${width} ${height3}"/>
-      </geometry>
-      <material name="orange"/>
-    </visual>
-    <inertial>
-      <origin xyz="0 0 ${height3/2 - axel_offset}" rpy="0 0 0"/>
-      <mass value="${mass}"/>
-      <inertia
-        ixx="${mass / 12.0 * (width*width + height3*height3)}" ixy="0.0" ixz="0.0"
-        iyy="${mass / 12.0 * (height3*height3 + width*width)}" iyz="0.0"
-        izz="${mass / 12.0 * (width*width + width*width)}"/>
-    </inertial>
-  </link>
-  <!-- Middle Link 2-->
-  <link name="${prefix}link3">
-    <collision>
-      <origin xyz="0 0 ${height2/2 - axel_offset}" rpy="0 0 0"/>
-      <geometry>
-        <box size="${width} ${width} ${height2}"/>
-      </geometry>
-    </collision>
-    <visual>
-      <origin xyz="0 0 ${height2/2 - axel_offset}" rpy="0 0 0"/>
-      <geometry>
-        <box size="${width} ${width} ${height2}"/>
-      </geometry>
-      <material name="red"/>
-    </visual>
+  <!-- Joint for Finger 1 Middle Segment -->
+  <joint name="${prefix}joint_finger1_middle" type="revolute">
+    <parent link="${prefix}finger1_base"/> <!-- Link to which the joint is connected -->
+    <child link="${prefix}finger1_middle"/> <!-- Link that the joint connects to -->
+    <!-- Joint origin and axis -->
+    <origin xyz="0 ${width} ${height1 - axel_offset}" rpy="0 0 0"/>
+    <axis xyz="0 1 0"/>
+    <!-- Joint dynamics (optional) -->
+    <dynamics damping="0.7"/>
+    <!-- Joint limits -->
+    <limit effort="100" velocity="1.0" lower="-3.14" upper="3.14"/>
+  </joint>
+  <!-- Finger 2 Base Link -->
+  <link name="${prefix}finger2_base">
+    <!-- Collision properties -->
+    <collision>
+      <origin xyz="0 0 ${height1/2}" rpy="0 0 0"/>
+      <geometry>
+        <box size="${width} ${width} ${height1}"/>
+      </geometry>
+    </collision>
+    <!-- Visual properties -->
+    <visual>
+      <origin xyz="0 0 ${height1/2}" rpy="0 0 0"/>
+      <geometry>
+        <box size="${width*4} ${width*10} ${height1}"/>
+      </geometry>
+      <material name="blue"/>
+    </visual>
+    <!-- Inertial properties -->
+    <inertial>
+      <origin xyz="0 0 ${height1/2}" rpy="0 0 0"/>
+      <mass value="${mass}"/>
+      <inertia
+        ixx="${mass / 12.0 * (width*width + height1*height1)}" ixy="0.0" ixz="0.0"
+        iyy="${mass / 12.0 * (height1*height1 + width*width)}" iyz="0.0"
+        izz="${mass / 12.0 * (width*width + width*width)}"/>
+    </inertial>
+  </link>
+  <!-- Joint for Finger 2 -->
+  <joint name="${prefix}joint_finger2" type="revolute">
+    <parent link="${prefix}base_link"/> <!-- Link to which the joint is connected -->
+    <child link="${prefix}finger2_base"/> <!-- Link that the joint connects to -->
+    <!-- Joint origin and axis -->
+    <origin xyz="0 -${width} ${height1 - axel_offset}" rpy="0 0 0"/>
+    <axis xyz="0 -1 0"/>
+    <!-- Joint dynamics (optional) -->
+    <dynamics damping="0.7"/>
+    <!-- Joint limits -->
+    <limit effort="100" velocity="1.0" lower="-3.14" upper="3.14"/>
+  </joint>
+  <!-- Finger 2 Middle Link -->
+  <link name="${prefix}finger2_middle">
+    <!-- Collision properties -->
+    <collision>
+      <origin xyz="0 0 ${height2/2 - axel_offset}" rpy="0 0 0"/>
+      <geometry>
+        <box size="${width} ${width} ${height2}"/>
+      </geometry>
+    </collision>
+    <!-- Visual properties -->
+    <visual>
+      <origin xyz="0 0 ${height2/2 - axel_offset}" rpy="0 0 0"/>
+      <geometry>
+        <box size="${width} ${width} ${height2}"/>
+      </geometry>
+      <material name="yellow"/>
+    </visual>
+    <!-- Inertial properties -->
     <inertial>
       <origin xyz="0 0 ${height2/2 - axel_offset}" rpy="0 0 0"/>
@@ -124,50 +181,94 @@
     </inertial>
   </link>
-  <joint name="${prefix}joint3" type="continuous">
-    <parent link="${prefix}base_link"/>
-    <child link="${prefix}link3"/>
+  <!-- Joint for Finger 2 Middle Segment -->
+  <joint name="${prefix}joint_finger2_middle" type="revolute">
+    <parent link="${prefix}finger2_base"/> <!-- Link to which the joint is connected -->
+    <child link="${prefix}finger2_middle"/> <!-- Link that the joint connects to -->
+    <!-- Joint origin and axis -->
+    <origin xyz="0 -${width} ${height1 - axel_offset}" rpy="0 0 0"/>
+    <axis xyz="0 -1 0"/>
+    <!-- Joint dynamics (optional) -->
+    <dynamics damping="0.7"/>
+    <!-- Joint limits -->
+    <limit effort="100" velocity="1.0" lower="-3.14" upper="3.14"/>
+  </joint>
+  <!-- Finger 3 Base Link -->
+  <link name="${prefix}finger3_base">
+    <!-- Collision properties -->
+    <collision>
+      <origin xyz="0 0 ${height1/2}" rpy="0 0 0"/>
+      <geometry>
+        <box size="${width} ${width} ${height1}"/>
+      </geometry>
+    </collision>
+    <!-- Visual properties -->
+    <visual>
+      <origin xyz="0 0 ${height1/2}" rpy="0 0 0"/>
+      <geometry>
+        <box size="${width*4} ${width*10} ${height1}"/>
+      </geometry>
+      <material name="blue"/>
+    </visual>
+    <!-- Inertial properties -->
+    <inertial>
+      <origin xyz="0 0 ${height1/2}" rpy="0 0 0"/>
+      <mass value="${mass}"/>
+      <inertia
+        ixx="${mass / 12.0 * (width*width + height1*height1)}" ixy="0.0" ixz="0.0"
+        iyy="${mass / 12.0 * (height1*height1 + width*width)}" iyz="0.0"
+        izz="${mass / 12.0 * (width*width + width*width)}"/>
+    </inertial>
+  </link>
+  <!-- Joint for Finger 3 -->
+  <joint name="${prefix}joint_finger3" type="revolute">
+    <parent link="${prefix}base_link"/> <!-- Link to which the joint is connected -->
+    <child link="${prefix}finger3_base"/> <!-- Link that the joint connects to -->
+    <!-- Joint origin and axis -->
     <origin xyz="0 ${width+0.5} ${height1 - axel_offset}" rpy="0 0 0"/>
     <axis xyz="0 1 0"/>
-    <dynamics damping="0.7"/>
-  </joint>
-  <!-- Top Link 2-->
-  <link name="${prefix}link4">
-    <collision>
-      <origin xyz="0 0 ${height3/2 - axel_offset}" rpy="0 0 0"/>
-      <geometry>
-        <box size="${width} ${width} ${height3}"/>
-      </geometry>
-    </collision>
-    <visual>
-      <origin xyz="0 0 ${height3/2 - axel_offset}" rpy="0 0 0"/>
-      <geometry>
-        <box size="${width} ${width} ${height3}"/>
-      </geometry>
-      <material name="orange"/>
-    </visual>
-    <inertial>
-      <origin xyz="0 0 ${height3/2 - axel_offset}" rpy="0 0 0"/>
-      <mass value="${mass}"/>
-      <inertia
-        ixx="${mass / 12.0 * (width*width + height3*height3)}" ixy="0.0" ixz="0.0"
-        iyy="${mass / 12.0 * (height3*height3 + width*width)}" iyz="0.0"
-        izz="${mass / 12.0 * (width*width + width*width)}"/>
-    </inertial>
-  </link>
-  <joint name="${prefix}joint4" type="continuous">
-    <parent link="${prefix}link3"/>
-    <child link="${prefix}link4"/>
-    <origin xyz="0 ${width} ${height2 - axel_offset}" rpy="0 0 0"/>
-    <axis xyz="0 1 0"/>
-    <dynamics damping="0.7"/>
-  </joint>
-  <joint name="${prefix}tool_joint" type="fixed">
-    <origin xyz="0 0 1" rpy="0 0 0" />
-    <parent link="${prefix}link3"/>
-    <child link="${prefix}tool_link" />
-  </joint>
-  <!-- Tool Link -->
-  <link name="${prefix}tool_link">
-  </link>
+    <!-- Joint dynamics (optional) -->
+    <dynamics damping="0.7"/>
+    <!-- Joint limits -->
+    <limit effort="100" velocity="1.0" lower="-3.14" upper="3.14"/>
+  </joint>
+  <!-- Finger 3 Middle Link -->
+  <link name="${prefix}finger3_middle">
+    <!-- Collision properties -->
+    <collision>
+      <origin xyz="0 0 ${height2/2 - axel_offset}" rpy="0 0 0"/>
+      <geometry>
+        <box size="${width} ${width} ${height2}"/>
+      </geometry>
+    </collision>
+    <!-- Visual properties -->
+    <visual>
+      <origin xyz="0 0 ${height2/2 - axel_offset}" rpy="0 0 0"/>
+      <geometry>
+        <box size="${width} ${width} ${height2}"/>
+      </geometry>
+      <material name="yellow"/>
+    </visual>
+    <!-- Inertial properties -->
+    <inertial>
+      <origin xyz="0 0 ${height2/2 - axel_offset}" rpy="0 0 0"/>
+      <mass value="${mass}"/>
+      <inertia
+        ixx="${mass / 12.0 * (width*width + height2*height2)}" ixy="0.0" ixz="0.0"
+        iyy="${mass / 12.0 * (height2*height2 + width*width)}" iyz="0.0"
+        izz="${mass / 12.0 * (width*width + width*width)}"/>
+    </inertial>
+  </link>
+  <!-- Joint for Finger 3 Middle Segment -->
+  <joint name="${prefix}joint_finger3_middle" type="revolute">
+    <parent link="${prefix}finger3_base"/> <!-- Link to which the joint is connected -->
+    <child link="${prefix}finger3_middle"/> <!-- Link that the joint connects to -->
+    <!-- Joint origin and axis -->
+    <origin xyz="0 ${width+0.5} ${height1 - axel_offset}" rpy="0 0 0"/>
+    <axis xyz="0 1 0"/>
+    <!-- Joint dynamics (optional) -->
+    <dynamics damping="0.7"/>
+    <!-- Joint limits -->
+    <limit effort="100" velocity="1.0" lower="-3.14" upper="3.14"/>
+  </joint>
   </xacro:macro>
 </robot>

File: src/ros2_control_hand/description/ros2_control/rrbot.ros2_control.xacro (robot description, xacro)
@@ -6,5 +6,5 @@
         <plugin>ros2_control_hand/CustomHardware</plugin>
       </hardware>
-      <joint name="${prefix}joint1">
+      <joint name="${prefix}finger1_joint">
         <command_interface name="position">
           <param name="min">-1</param>
@@ -13,5 +13,5 @@
         <state_interface name="position"/>
       </joint>
-      <joint name="${prefix}joint2">
+      <joint name="${prefix}finger1_middle_joint">
         <command_interface name="position">
           <param name="min">-1</param>
@@ -20,5 +20,5 @@
         <state_interface name="position"/>
       </joint>
-      <joint name="${prefix}joint3">
+      <joint name="${prefix}finger2_joint">
         <command_interface name="position">
           <param name="min">-1</param>
@@ -27,5 +27,19 @@
         <state_interface name="position"/>
       </joint>
-      <joint name="${prefix}joint4">
+      <joint name="${prefix}finger2_middle_joint">
+        <command_interface name="position">
+          <param name="min">-1</param>
+          <param name="max">1</param>
+        </command_interface>
+        <state_interface name="position"/>
+      </joint>
+      <joint name="${prefix}finger3_joint">
+        <command_interface name="position">
+          <param name="min">-1</param>
+          <param name="max">1</param>
+        </command_interface>
+        <state_interface name="position"/>
+      </joint>
+      <joint name="${prefix}finger3_middle_joint">
         <command_interface name="position">
           <param name="min">-1</param>
