Commit message: ajout main

File: install/ros2_control_demo_description/share/ros2_control_demo_description/rrbot/urdf/rrbot_description.urdf.xacro (robot description, xacro)
@@ -271,4 +271,160 @@
     <limit effort="100" velocity="1.0" lower="-3.14" upper="3.14"/>
   </joint>
+    <!-- Finger 4 Base Link -->
+  <link name="${prefix}finger4_base">
+    <!-- Collision properties -->
+    <collision>
+      <origin xyz="0 0 ${height1/2}" rpy="0 0 0"/>
+      <geometry>
+        <box size="${width} ${width} ${height1}"/>
+      </geometry>
+    </collision>
+    <!-- Visual properties -->
+    <visual>
+      <origin xyz="0 0 ${height1/2}" rpy="0 0 0"/>
+      <geometry>
+        <box size="${width*4} ${width*10} ${height1}"/>
+      </geometry>
+      <material name="blue"/>
+    </visual>
+    <!-- Inertial properties -->
+    <inertial>
+      <origin xyz="0 0 ${height1/2}" rpy="0 0 0"/>
+      <mass value="${mass}"/>
+      <inertia
+        ixx="${mass / 12.0 * (width*width + height1*height1)}" ixy="0.0" ixz="0.0"
+        iyy="${mass / 12.0 * (height1*height1 + width*width)}" iyz="0.0"
+        izz="${mass / 12.0 * (width*width + width*width)}"/>
+    </inertial>
+  </link>
+  <!-- Joint for Finger 4 -->
+  <joint name="${prefix}joint_finger4" type="revolute">
+    <parent link="${prefix}base_link"/> <!-- Link to which the joint is connected -->
+    <child link="${prefix}finger4_base"/> <!-- Link that the joint connects to -->
+    <!-- Joint origin and axis -->
+    <origin xyz="0 ${width*2} ${height1 - axel_offset}" rpy="0 0 0"/>
+    <axis xyz="0 1 0"/>
+    <!-- Joint dynamics (optional) -->
+    <dynamics damping="0.7"/>
+    <!-- Joint limits -->
+    <limit effort="100" velocity="1.0" lower="-3.14" upper="3.14"/>
+  </joint>
+  <!-- Finger 4 Middle Link -->
+  <link name="${prefix}finger4_middle">
+    <!-- Collision properties -->
+    <collision>
+      <origin xyz="0 0 ${height2/2 - axel_offset}" rpy="0 0 0"/>
+      <geometry>
+        <box size="${width} ${width} ${height2}"/>
+      </geometry>
+    </collision>
+    <!-- Visual properties -->
+    <visual>
+      <origin xyz="0 0 ${height2/2 - axel_offset}" rpy="0 0 0"/>
+      <geometry>
+        <box size="${width} ${width} ${height2}"/>
+      </geometry>
+      <material name="yellow"/>
+    </visual>
+    <!-- Inertial properties -->
+    <inertial>
+      <origin xyz="0 0 ${height2/2 - axel_offset}" rpy="0 0 0"/>
+      <mass value="${mass}"/>
+      <inertia
+        ixx="${mass / 12.0 * (width*width + height2*height2)}" ixy="0.0" ixz="0.0"
+        iyy="${mass / 12.0 * (height2*height2 + width*width)}" iyz="0.0"
+        izz="${mass / 12.0 * (width*width + width*width)}"/>
+    </inertial>
+  </link>
+  <!-- Joint for Finger 4 Middle Segment -->
+  <joint name="${prefix}joint_finger4_middle" type="revolute">
+    <parent link="${prefix}finger4_base"/> <!-- Link to which the joint is connected -->
+    <child link="${prefix}finger4_middle"/> <!-- Link that the joint connects to -->
+    <!-- Joint origin and axis -->
+    <origin xyz="0 ${width*2} ${height1 - axel_offset}" rpy="0 0 0"/>
+    <axis xyz="0 1 0"/>
+    <!-- Joint dynamics (optional) -->
+    <dynamics damping="0.7"/>
+    <!-- Joint limits -->
+    <limit effort="100" velocity="1.0" lower="-3.14" upper="3.14"/>
+  </joint>
+    <!-- Thumb Base Link -->
+  <link name="${prefix}thumb_base">
+    <!-- Collision properties -->
+    <collision>
+      <origin xyz="0 0 ${height1/2}" rpy="0 0 0"/>
+      <geometry>
+        <box size="${width} ${width} ${height1}"/>
+      </geometry>
+    </collision>
+    <!-- Visual properties -->
+    <visual>
+      <origin xyz="0 0 ${height1/2}" rpy="0 0 0"/>
+      <geometry>
+        <box size="${width*4} ${width*10} ${height1}"/>
+      </geometry>
+      <material name="blue"/>
+    </visual>
+    <!-- Inertial properties -->
+    <inertial>
+      <origin xyz="0 0 ${height1/2}" rpy="0 0 0"/>
+      <mass value="${mass}"/>
+      <inertia
+        ixx="${mass / 12.0 * (width*width + height1*height1)}" ixy="0.0" ixz="0.0"
+        iyy="${mass / 12.0 * (height1*height1 + width*width)}" iyz="0.0"
+        izz="${mass / 12.0 * (width*width + width*width)}"/>
+    </inertial>
+  </link>
+  <!-- Joint for Thumb -->
+  <joint name="${prefix}joint_thumb" type="revolute">
+    <parent link="${prefix}base_link"/> <!-- Link to which the joint is connected -->
+    <child link="${prefix}thumb_base"/> <!-- Link that the joint connects to -->
+    <!-- Joint origin and axis -->
+    <origin xyz="0 -${width*2} ${height1 - axel_offset}" rpy="0 0 0"/>
+    <axis xyz="0 -1 0"/>
+    <!-- Joint dynamics (optional) -->
+    <dynamics damping="0.7"/>
+    <!-- Joint limits -->
+    <limit effort="100" velocity="1.0" lower="-3.14" upper="3.14"/>
+  </joint>
+  <!-- Thumb Middle Link -->
+  <link name="${prefix}thumb_middle">
+    <!-- Collision properties -->
+    <collision>
+      <origin xyz="0 0 ${height2/2 - axel_offset}" rpy="0 0 0"/>
+      <geometry>
+        <box size="${width} ${width} ${height2}"/>
+      </geometry>
+    </collision>
+    <!-- Visual properties -->
+    <visual>
+      <origin xyz="0 0 ${height2/2 - axel_offset}" rpy="0 0 0"/>
+      <geometry>
+        <box size="${width} ${width} ${height2}"/>
+      </geometry>
+      <material name="yellow"/>
+    </visual>
+    <!-- Inertial properties -->
+    <inertial>
+      <origin xyz="0 0 ${height2/2 - axel_offset}" rpy="0 0 0"/>
+      <mass value="${mass}"/>
+      <inertia
+        ixx="${mass / 12.0 * (width*width + height2*height2)}" ixy="0.0" ixz="0.0"
+        iyy="${mass / 12.0 * (height2*height2 + width*width)}" iyz="0.0"
+        izz="${mass / 12.0 * (width*width + width*width)}"/>
+    </inertial>
+  </link>
+  <!-- Joint for Thumb Middle Segment -->
+  <joint name="${prefix}joint_thumb_middle" type="revolute">
+    <parent link="${prefix}thumb_base"/> <!-- Link to which the joint is connected -->
+    <child link="${prefix}thumb_middle"/> <!-- Link that the joint connects to -->
+    <!-- Joint origin and axis -->
+    <origin xyz="0 -${width*2} ${height1 - axel_offset}" rpy="0 0 0"/>
+    <axis xyz="0 -1 0"/>
+    <!-- Joint dynamics (optional) -->
+    <dynamics damping="0.7"/>
+    <!-- Joint limits -->
+    <limit effort="100" velocity="1.0" lower="-3.14" upper="3.14"/>
+  </joint>
   </xacro:macro>
 </robot>

File: src/ros2_control_hand/description/ros2_control/rrbot.ros2_control.xacro (robot description, xacro)
@@ -6,5 +6,5 @@
         <plugin>ros2_control_hand/CustomHardware</plugin>
       </hardware>
-      <joint name="${prefix}finger1_joint">
+      <joint name="{$prefix}joint_finger_1_base">
         <command_interface name="position">
           <param name="min">-1</param>
@@ -13,5 +13,11 @@
         <state_interface name="position"/>
       </joint>
-      <joint name="${prefix}finger1_middle_joint">
+      <joint name="{$prefix}joint_finger_1_top">
+        <command_interface name="position">
+          <param name="min">-1</param>
+          <param name="max">1</param>
+        </command_interface>
+        <state_interface name="position"/>
+      </joint><joint name="{$prefix}link_finger_2_base">
         <command_interface name="position">
           <param name="min">-1</param>
@@ -20,5 +26,5 @@
         <state_interface name="position"/>
       </joint>
-      <joint name="${prefix}finger2_joint">
+      <joint name="{$prefix}joint_finger_2_top">
         <command_interface name="position">
           <param name="min">-1</param>
@@ -27,5 +33,5 @@
         <state_interface name="position"/>
       </joint>
-      <joint name="${prefix}finger2_middle_joint">
+      <joint name="{$prefix}joint_finger_3_base">
         <command_interface name="position">
           <param name="min">-1</param>
@@ -34,5 +40,5 @@
         <state_interface name="position"/>
       </joint>
-      <joint name="${prefix}finger3_joint">
+      <joint name="{$prefix}joint_finger_3_top">
         <command_interface name="position">
           <param name="min">-1</param>
@@ -41,5 +47,26 @@
         <state_interface name="position"/>
       </joint>
-      <joint name="${prefix}finger3_middle_joint">
+      <joint name="{$prefix}joint_finger_4_base">
+        <command_interface name="position">
+          <param name="min">-1</param>
+          <param name="max">1</param>
+        </command_interface>
+        <state_interface name="position"/>
+      </joint>
+      <joint name="{$prefix}joint_finger_4_top">
+        <command_interface name="position">
+          <param name="min">-1</param>
+          <param name="max">1</param>
+        </command_interface>
+        <state_interface name="position"/>
+      </joint>
+      <joint name="{$prefix}joint_thumb_base">
+        <command_interface name="position">
+          <param name="min">-1</param>
+          <param name="max">1</param>
+        </command_interface>
+        <state_interface name="position"/>
+      </joint>
+      <joint name="{$prefix}joint_thumb_top">
         <command_interface name="position">
           <param name="min">-1</param>

File: src/ros2_control_hand/description/urdf/rrbot.urdf.xacro (robot description, xacro)
@@ -8,5 +8,6 @@
   <xacro:arg name="prefix" default="" />
   <!-- Import RRBot macro -->
-  <xacro:include filename="$(find ros2_control_demo_description)/rrbot/urdf/rrbot_description.urdf.xacro" />
+  <!--xacro:include filename="$(find ros2_control_demo_description)/rrbot/urdf/rrbot_description.urdf.xacro" /-->
+  <xacro:include filename="$(find hand_urdf)/urdf/hand_urdf.urdf" />
   <!-- Import Rviz colors -->
   <xacro:include filename="$(find ros2_control_demo_description)/rrbot/urdf/rrbot.materials.xacro" />
