Commit message: f

File: install/dexhand_description/share/dexhand_description/urdf/ros2_control_hand.xacro (robot description, xacro)
@@ -3,7 +3,162 @@
     <ros2_control name="dexhand" type="system">
         <hardware>
-        <plugin>ros2_control_hand/CustomHardware</plugin>
+            <plugin>ros2_control_hand/CustomHardware</plugin>
         </hardware>
+        <joint name="index_knuckle">
+            <command_interface name="position">
+                <param name="min">-1</param>
+                <param name="max">1</param>
+            </command_interface>
+            <state_interface name="position"/>
+        </joint>
+        <joint name="index_pitch">
+            <command_interface name="position">
+                <param name="min">-1</param>
+                <param name="max">1</param>
+            </command_interface>
+            <state_interface name="position"/>
+        </joint>
+        <joint name="index_tip">
+            <command_interface name="position">
+                <param name="min">-1</param>
+                <param name="max">1</param>
+            </command_interface>
+            <state_interface name="position"/>
+        </joint>
+        <joint name="index_yaw">
+            <command_interface name="position">
+                <param name="min">-1</param>
+                <param name="max">1</param>
+            </command_interface>
+            <state_interface name="position"/>
+        </joint>
+        <joint name="middle_knuckle">
+            <command_interface name="position">
+                <param name="min">-1</param>
+                <param name="max">1</param>
+            </command_interface>
+            <state_interface name="position"/>
+        </joint>
+        <joint name="middle_pitch">
+            <command_interface name="position">
+                <param name="min">-1</param>
+                <param name="max">1</param>
+            </command_interface>
+            <state_interface name="position"/>
+        </joint>
+        <joint name="middle_tip">
+            <command_interface name="position">
+                <param name="min">-1</param>
+                <param name="max">1</param>
+            </command_interface>
+            <state_interface name="position"/>
+        </joint>
+        <joint name="middle_yaw">
+            <command_interface name="position">
+                <param name="min">-1</param>
+                <param name="max">1</param>
+            </command_interface>
+            <state_interface name="position"/>
+        </joint>
+        <!-- Continuez ici en ajoutant les autres joints triés par ordre alphabétique -->
+        <joint name="pinky_knuckle">
+            <command_interface name="position">
+                <param name="min">-1</param>
+                <param name="max">1</param>
+            </command_interface>
+            <state_interface name="position"/>
+        </joint>
+        <joint name="pinky_pitch">
+            <command_interface name="position">
+                <param name="min">-1</param>
+                <param name="max">1</param>
+            </command_interface>
+            <state_interface name="position"/>
+        </joint>
+        <joint name="pinky_tip">
+            <command_interface name="position">
+                <param name="min">-1</param>
+                <param name="max">1</param>
+            </command_interface>
+            <state_interface name="position"/>
+        </joint>
+        <joint name="pinky_yaw">
+            <command_interface name="position">
+                <param name="min">-1</param>
+                <param name="max">1</param>
+            </command_interface>
+            <state_interface name="position"/>
+        </joint>
+        <joint name="ring_knuckle">
+            <command_interface name="position">
+                <param name="min">-1</param>
+                <param name="max">1</param>
+            </command_interface>
+            <state_interface name="position"/>
+        </joint>
+        <joint name="ring_pitch">
+            <command_interface name="position">
+                <param name="min">-1</param>
+                <param name="max">1</param>
+            </command_interface>
+            <state_interface name="position"/>
+        </joint>
+        <joint name="ring_tip">
+            <command_interface name="position">
+                <param name="min">-1</param>
+                <param name="max">1</param>
+            </command_interface>
+            <state_interface name="position"/>
+        </joint>
+        <joint name="ring_yaw">
+            <command_interface name="position">
+                <param name="min">-1</param>
+                <param name="max">1</param>
+            </command_interface>
+            <state_interface name="position"/>
+        </joint>
+        <joint name="thumb_knuckle">
+            <command_interface name="position">
+                <param name="min">-1</param>
+                <param name="max">1</param>
+            </command_interface>
+            <state_interface name="position"/>
+        </joint>
+        <joint name="thumb_pitch">
+            <command_interface name="position">
+                <param name="min">-1</param>
+                <param name="max">1</param>
+            </command_interface>
+            <state_interface name="position"/>
+        </joint>
+        <joint name="thumb_roll">
+            <command_interface name="position">
+                <param name="min">-1</param>
+                <param name="max">1</param>
+            </command_interface>
+            <state_interface name="position"/>
+        </joint>
+        <joint name="thumb_tip">
+            <command_interface name="position">
+                <param name="min">-1</param>
+                <param name="max">1</param>
+            </command_interface>
+            <state_interface name="position"/>
+        </joint>
+        <joint name="thumb_yaw">
+            <command_interface name="position">
+                <param name="min">-1</param>
+                <param name="max">1</param>
+            </command_interface>
+            <state_interface name="position"/>
+        </joint>
         <joint name="wrist_pitch_lower">
+            <command_interface name="position">
+                <param name="min">-1</param>
+                <param name="max">1</param>
+            </command_interface>
+            <state_interface name="position"/>
+        </joint>
+        <joint name="wrist_pitch_upper">
             <command_interface name="position">
                 <param name="min">-1</param>
@@ -19,158 +174,4 @@
             <state_interface name="position"/>
         </joint>
-        <joint name="wrist_pitch_upper">
-            <command_interface name="position">
-                <param name="min">-1</param>
-                <param name="max">1</param>
-            </command_interface>
-            <state_interface name="position"/>
-        </joint>
-        <joint name="index_yaw">
-            <command_interface name="position">
-                <param name="min">-1</param>
-                <param name="max">1</param>
-            </command_interface>
-            <state_interface name="position"/>
-        </joint>
-        <joint name="middle_yaw">
-            <command_interface name="position">
-                <param name="min">-1</param>
-                <param name="max">1</param>
-            </command_interface>
-            <state_interface name="position"/>
-        </joint>
-        <joint name="ring_yaw">
-            <command_interface name="position">
-                <param name="min">-1</param>
-                <param name="max">1</param>
-            </command_interface>
-            <state_interface name="position"/>
-        </joint>
-        <joint name="pinky_yaw">
-            <command_interface name="position">
-                <param name="min">-1</param>
-                <param name="max">1</param>
-            </command_interface>
-            <state_interface name="position"/>
-        </joint>
-        <joint name="index_pitch">
-            <command_interface name="position">
-                <param name="min">-1</param>
-                <param name="max">1</param>
-            </command_interface>
-            <state_interface name="position"/>
-        </joint>
-        <joint name="index_knuckle">
-            <command_interface name="position">
-                <param name="min">-1</param>
-                <param name="max">1</param>
-            </command_interface>
-            <state_interface name="position"/>
-        </joint>
-        <joint name="index_tip">
-            <command_interface name="position">
-                <param name="min">-1</param>
-                <param name="max">1</param>
-            </command_interface>
-            <state_interface name="position"/>
-        </joint>
-        <joint name="middle_pitch">
-            <command_interface name="position">
-                <param name="min">-1</param>
-                <param name="max">1</param>
-            </command_interface>
-            <state_interface name="position"/>
-        </joint>
-        <joint name="middle_knuckle">
-            <command_interface name="position">
-                <param name="min">-1</param>
-                <param name="max">1</param>
-            </command_interface>
-            <state_interface name="position"/>
-        </joint>
-        <joint name="middle_tip">
-            <command_interface name="position">
-                <param name="min">-1</param>
-                <param name="max">1</param>
-            </command_interface>
-            <state_interface name="position"/>
-        </joint>
-        <joint name="ring_pitch">
-            <command_interface name="position">
-                <param name="min">-1</param>
-                <param name="max">1</param>
-            </command_interface>
-            <state_interface name="position"/>
-        </joint>
-        <joint name="ring_knuckle">
-            <command_interface name="position">
-                <param name="min">-1</param>
-                <param name="max">1</param>
-            </command_interface>
-            <state_interface name="position"/>
-        </joint>
-        <joint name="ring_tip">
-            <command_interface name="position">
-                <param name="min">-1</param>
-                <param name="max">1</param>
-            </command_interface>
-            <state_interface name="position"/>
-        </joint>
-        <joint name="pinky_pitch">
-            <command_interface name="position">
-                <param name="min">-1</param>
-                <param name="max">1</param>
-            </command_interface>
-            <state_interface name="position"/>
-        </joint>
-        <joint name="pinky_knuckle">
-            <command_interface name="position">
-                <param name="min">-1</param>
-                <param name="max">1</param>
-            </command_interface>
-            <state_interface name="position"/>
-        </joint>
-        <joint name="pinky_tip">
-            <command_interface name="position">
-                <param name="min">-1</param>
-                <param name="max">1</param>
-            </command_interface>
-            <state_interface name="position"/>
-        </joint>
-        <joint name="thumb_yaw">
-            <command_interface name="position">
-                <param name="min">-1</param>
-                <param name="max">1</param>
-            </command_interface>
-            <state_interface name="position"/>
-        </joint>
-        <joint name="thumb_roll">
-            <command_interface name="position">
-                <param name="min">-1</param>
-                <param name="max">1</param>
-            </command_interface>
-            <state_interface name="position"/>
-        </joint>
-        <joint name="thumb_pitch">
-            <command_interface name="position">
-                <param name="min">-1</param>
-                <param name="max">1</param>
-            </command_interface>
-            <state_interface name="position"/>
-        </joint>
-        <joint name="thumb_knuckle">
-            <command_interface name="position">
-                <param name="min">-1</param>
-                <param name="max">1</param>
-            </command_interface>
-            <state_interface name="position"/>
-        </joint>
-        <joint name="thumb_tip">
-            <command_interface name="position">
-                <param name="min">-1</param>
-                <param name="max">1</param>
-            </command_interface>
-            <state_interface name="position"/>
-        </joint>
     </ros2_control>
 </robot>

Commit message: got first letter of joint

File: install/dexhand_description/share/dexhand_description/urdf/ros2_control_hand.xacro (robot description, xacro)
@@ -5,5 +5,5 @@
             <plugin>ros2_control_hand/CustomHardware</plugin>
         </hardware>
-        <joint name="index_knuckle">
+        <joint name="index_yaw________">
             <command_interface name="position">
                 <param name="min">-1</param>
@@ -12,5 +12,5 @@
             <state_interface name="position"/>
         </joint>
-        <joint name="index_pitch">
+        <joint name="middle_knuckle___">
             <command_interface name="position">
                 <param name="min">-1</param>
@@ -19,5 +19,5 @@
             <state_interface name="position"/>
         </joint>
-        <joint name="index_tip">
+        <joint name="index_tip________">
             <command_interface name="position">
                 <param name="min">-1</param>
@@ -26,5 +26,5 @@
             <state_interface name="position"/>
         </joint>
-        <joint name="index_yaw">
+        <joint name="middle_yaw_______">
             <command_interface name="position">
                 <param name="min">-1</param>
@@ -33,5 +33,5 @@
             <state_interface name="position"/>
         </joint>
-        <joint name="middle_knuckle">
+        <joint name="pinky_knuckle____">
             <command_interface name="position">
                 <param name="min">-1</param>
@@ -40,5 +40,5 @@
             <state_interface name="position"/>
         </joint>
-        <joint name="middle_pitch">
+        <joint name="pinky_pitch______">
             <command_interface name="position">
                 <param name="min">-1</param>
@@ -47,5 +47,5 @@
             <state_interface name="position"/>
         </joint>
-        <joint name="middle_tip">
+        <joint name="index_pitch______">
             <command_interface name="position">
                 <param name="min">-1</param>
@@ -54,5 +54,5 @@
             <state_interface name="position"/>
         </joint>
-        <joint name="middle_yaw">
+        <joint name="wrist_yaw________">
             <command_interface name="position">
                 <param name="min">-1</param>
@@ -62,5 +62,5 @@
         </joint>
         <!-- Continuez ici en ajoutant les autres joints triés par ordre alphabétique -->
-        <joint name="pinky_knuckle">
+        <joint name="middle_tip_______">
             <command_interface name="position">
                 <param name="min">-1</param>
@@ -69,82 +69,5 @@
             <state_interface name="position"/>
         </joint>
-        <joint name="pinky_pitch">
-            <command_interface name="position">
-                <param name="min">-1</param>
-                <param name="max">1</param>
-            </command_interface>
-            <state_interface name="position"/>
-        </joint>
-        <joint name="pinky_tip">
-            <command_interface name="position">
-                <param name="min">-1</param>
-                <param name="max">1</param>
-            </command_interface>
-            <state_interface name="position"/>
-        </joint>
-        <joint name="pinky_yaw">
-            <command_interface name="position">
-                <param name="min">-1</param>
-                <param name="max">1</param>
-            </command_interface>
-            <state_interface name="position"/>
-        </joint>
-        <joint name="ring_knuckle">
-            <command_interface name="position">
-                <param name="min">-1</param>
-                <param name="max">1</param>
-            </command_interface>
-            <state_interface name="position"/>
-        </joint>
-        <joint name="ring_pitch">
-            <command_interface name="position">
-                <param name="min">-1</param>
-                <param name="max">1</param>
-            </command_interface>
-            <state_interface name="position"/>
-        </joint>
-        <joint name="ring_tip">
-            <command_interface name="position">
-                <param name="min">-1</param>
-                <param name="max">1</param>
-            </command_interface>
-            <state_interface name="position"/>
-        </joint>
-        <joint name="ring_yaw">
-            <command_interface name="position">
-                <param name="min">-1</param>
-                <param name="max">1</param>
-            </command_interface>
-            <state_interface name="position"/>
-        </joint>
-        <joint name="thumb_knuckle">
-            <command_interface name="position">
-                <param name="min">-1</param>
-                <param name="max">1</param>
-            </command_interface>
-            <state_interface name="position"/>
-        </joint>
-        <joint name="thumb_pitch">
-            <command_interface name="position">
-                <param name="min">-1</param>
-                <param name="max">1</param>
-            </command_interface>
-            <state_interface name="position"/>
-        </joint>
-        <joint name="thumb_roll">
-            <command_interface name="position">
-                <param name="min">-1</param>
-                <param name="max">1</param>
-            </command_interface>
-            <state_interface name="position"/>
-        </joint>
-        <joint name="thumb_tip">
-            <command_interface name="position">
-                <param name="min">-1</param>
-                <param name="max">1</param>
-            </command_interface>
-            <state_interface name="position"/>
-        </joint>
-        <joint name="thumb_yaw">
+        <joint name="wrist_pitch_upper">
             <command_interface name="position">
                 <param name="min">-1</param>
@@ -160,5 +83,5 @@
             <state_interface name="position"/>
         </joint>
-        <joint name="wrist_pitch_upper">
+        <joint name="pinky_tip________">
             <command_interface name="position">
                 <param name="min">-1</param>
@@ -167,5 +90,82 @@
             <state_interface name="position"/>
         </joint>
-        <joint name="wrist_yaw">
+        <joint name="thumb_knuckle____">
+            <command_interface name="position">
+                <param name="min">-1</param>
+                <param name="max">1</param>
+            </command_interface>
+            <state_interface name="position"/>
+        </joint>
+        <joint name="middle_pitch_____">
+            <command_interface name="position">
+                <param name="min">-1</param>
+                <param name="max">1</param>
+            </command_interface>
+            <state_interface name="position"/>
+        </joint>
+        <joint name="ring_pitch_______">
+            <command_interface name="position">
+                <param name="min">-1</param>
+                <param name="max">1</param>
+            </command_interface>
+            <state_interface name="position"/>
+        </joint>
+        <joint name="ring_knuckle_____">
+            <command_interface name="position">
+                <param name="min">-1</param>
+                <param name="max">1</param>
+            </command_interface>
+            <state_interface name="position"/>
+        </joint>
+        <joint name="thumb_tip________">
+            <command_interface name="position">
+                <param name="min">-1</param>
+                <param name="max">1</param>
+            </command_interface>
+            <state_interface name="position"/>
+        </joint>
+        <joint name="thumb_yaw________">
+            <command_interface name="position">
+                <param name="min">-1</param>
+                <param name="max">1</param>
+            </command_interface>
+            <state_interface name="position"/>
+        </joint>
+        <joint name="thumb_roll_______">
+            <command_interface name="position">
+                <param name="min">-1</param>
+                <param name="max">1</param>
+            </command_interface>
+            <state_interface name="position"/>
+        </joint>
+        <joint name="thumb_pitch______">
+            <command_interface name="position">
+                <param name="min">-1</param>
+                <param name="max">1</param>
+            </command_interface>
+            <state_interface name="position"/>
+        </joint>
+        <joint name="ring_yaw_________">
+            <command_interface name="position">
+                <param name="min">-1</param>
+                <param name="max">1</param>
+            </command_interface>
+            <state_interface name="position"/>
+        </joint>
+        <joint name="ring_tip_________">
+            <command_interface name="position">
+                <param name="min">-1</param>
+                <param name="max">1</param>
+            </command_interface>
+            <state_interface name="position"/>
+        </joint>
+        <joint name="index_knuckle____">
+            <command_interface name="position">
+                <param name="min">-1</param>
+                <param name="max">1</param>
+            </command_interface>
+            <state_interface name="position"/>
+        </joint>
+        <joint name="pinky_yaw________">
             <command_interface name="position">
                 <param name="min">-1</param>
